File: Peripherals.kicad_sch (KiCad schematic)
At the start: 19 parts, among them J3 0532610271, J6 0532610671, U4 DRV2605LDGS, U5 BNO055, U6 M20048-1

Commit message: Updated board outline to version 004
Other:
- note added: "<30 μA"
- note added: "ADDR_{(7)} = 0x28"
- note added: "ADDR_{(7)} = 0x5A"
- note added: "COMPASS HMC5883L ADDR_{(7)} = 0x1E"
- note removed: "0x28"
Changed lines of the file:
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@@
+		)
+	)
+	(text "ADDR_{(7)} = 0x5A"
+		(exclude_from_sim no)
+		(at 52.578 161.544 0)
+		(effects
+			(font
+				(size 1 1)
+				(thickness 0.1588)
+				(color 0 132 132 1)
+			)
 		)
 	)
@@
 		)
 	)
-	(text "0x28"
+	(text "ADDR_{(7)} = 0x28"
 		(exclude_from_sim no)
-		(at 168.91 145.288 0)
+		(at 151.638 161.544 0)
 		(effects
 			(font
 				(size 1 1)
 				(thickness 0.1588)
+				(color 0 132 132 1)
 			)
 		)
@@
 		)
 	)
+	(text "COMPASS HMC5883L\nADDR_{(7)} = 0x1E"
+		(exclude_from_sim no)
+		(at 235.204 89.408 0)
+		(effects
+			(font
+				(size 1 1)
+				(thickness 0.1588)
+				(color 0 132 132 1)
+			)
+			(justify right)
+		)
+	)
 	(text "GPS Options"
 		(exclude_from_sim no)
@@
 		)
 	)
+	(text "<30 μA"
+		(exclude_from_sim no)
+		(at 61.976 70.104 0)
+		(effects
+			(font
+				(size 1 1)
+				(color 132 0 132 1)
+			)
+			(justify left)
+		)
+	)

Commit message: Lots of board layout
Parts:
- added C19: 1u, Capacitor_SMD:C_0603_1608Metric, symbol Device:C
- added J5: B8B-PH-SM4-TB, Connector_JST:JST_PH_B8B-PH-SM4-TB_1x08-1MP_P2.00mm_Vertical, symbol Connector_Generic_MountingPin:Conn_01x08_MountingPin
Connections:
- net +3.3V: now also C19.1, J5.1 (Pin_1)
- net GND: now also C19.2, J5.2 (Pin_2), J5.MP (MountPin)
- new net DISP_DC: J5.6 (Pin_6)
- new net DISP_PWM_BL: J5.8 (Pin_8)
- new net DISP_~{RST}: J5.7 (Pin_7)
- new net SPI_MOSI: J5.3 (Pin_3)
- new net SPI_SCK: J5.4 (Pin_4)
- new net SPI_~{CS0_DISP}: J5.5 (Pin_5)
Other:
- note added: "Display Connector"
- note added: "Waveshare 1.28" 240x240 px LCD 19192"
- moved on the sheet: C10, C11, C13, C14, C15, C16, C9, J3, J6, L1, R19, R20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

Commit message: More layout and sch updates, ready for final review.
Parts:
- J5: MPN (none) -> B8B-PH-SM4-TB
- J6: MPN (none) -> 0532610671
- U4: MPN (none) -> DRV2605LDGS
- U5: MPN (none) -> BNO055
Changed lines of the file:
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@@
 	(title_block
 		(title "${TITLE}")
-		(date "2025-03-23")
+		(date "2025-04-05")
 		(rev "${REVISION}")
 		(company "J. MENDEL")
@@
 			)
 		)
+		(property "MPN" "0532610671"
+			(at 184.15 54.61 0)
+			(effects
+				(font
+					(size 1.27 1.27)
+				)
+				(hide yes)
+			)
+		)
 		(pin "4"
 		)
@@
 			)
 		)
+		(property "MPN" "BNO055"
+			(at 162.56 130.81 0)
+			(effects
+				(font
+					(size 1.27 1.27)
+				)
+				(hide yes)
+			)
+		)
 		(pin "11"
 		)
@@
 			)
 		)
-		(property "Datasheet" "~"
+		(property "Datasheet" "https://search.murata.co.jp/Ceramy/image/img/P02/JELF243B-9117.pdf"
 			(at 118.11 40.64 0)
 			(effects
@@
 			)
 		)
+		(property "MPN" "DRV2605LDGS"
+			(at 53.34 129.54 0)
+			(effects
+				(font
+					(size 1.27 1.27)
+				)
+				(hide yes)
+			)
+		)
 		(pin "5"
 		)
@@
 			(at 243.84 40.64 0)
 			(effects
+				(font
+					(size 1.27 1.27)
+				)
+				(hide yes)
+			)
+		)
+		(property "MPN" "B8B-PH-SM4-TB"
+			(at 243.84 40.64 0)
+			(effects

Commit message: For design review X01-001 Ammendment: Changed ALL VIAS to 0.3/0.55 to reduce fab cost. Signed-off-by: James Mendel <jrm.mendel@gmail.com>
Parts:
- C10, C11, C19, C9: MPN (none) -> CL10A105KO8NNNC
- C13, C14: MPN (none) -> CL10B104KO8NNNC
- C15, C16: MPN (none) -> CL10C220JB8NNNC
- L1: footprint Inductor_SMD:L_0402_1005Metric -> Inductor_SMD:L_0603_1608Metric; MPN LQG15WZ1N8C02D -> HK16081N8S-T
- R19, R20: MPN (none) -> RC0603FR-0710KL
- R24, R25: footprint Resistor_SMD:R_0402_1005Metric -> Resistor_SMD:R_0603_1608Metric; MPN (none) -> RC0603FR-070RL
Changed lines of the file:
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@@
 			)
 		)
+		(property "MPN" "CL10A105KO8NNNC"
+			(at 60.96 115.57 0)
+			(effects
+				(font
+					(size 1.27 1.27)
+				)
+				(hide yes)
+			)
+		)
 		(pin "1"
 		)
@@
 			)
 		)
+		(property "MPN" "CL10A105KO8NNNC"
+			(at 182.88 149.86 0)
+			(effects
+				(font
+					(size 1.27 1.27)
+				)
+			)
+		)
 		(pin "1"
 		)
@@
 			)
 		)
-		(property "Datasheet" "~"
+		(property "Datasheet" "https://www.lcsc.com/datasheet/lcsc_datasheet_2304140030_YAGEO-RC0603FR-071KL_C22548.pdf"
 			(at 137.16 113.03 0)
 			(effects
@@
 			)
 		)
+		(property "MPN" "RC0603FR-0710KL"
+			(at 137.16 113.03 0)
+			(effects
+				(font
+					(size 1.27 1.27)
+				)
+				(hide yes)
+			)
+		)
 		(pin "1"
 		)
@@
 			)
 		)
+		(property "MPN" "CL10B104KO8NNNC"
+			(at 186.69 114.3 0)
+			(effects
+				(font
+					(size 1.27 1.27)
+				)
+				(hide yes)
+			)
+		)
 		(pin "1"
 		)
@@
 			)
 		)
+		(property "MPN" "CL10C220JB8NNNC"
+			(at 57.15 50.8 0)
+			(effects
+				(font
+					(size 1.27 1.27)
+				)
+				(hide yes)
+			)
+		)
 		(pin "1"
 		)
@@
 			)
 		)
+		(property "MPN" "CL10A105KO8NNNC"
+			(at 76.2 139.7 0)
+			(effects
+				(font
+					(size 1.27 1.27)
+				)
+				(hide yes)
+			)
+		)
 		(pin "1"
 		)
@@
 			)
 		)
-		(property "Footprint" "Resistor_SMD:R_0402_1005Metric"
+		(property "Footprint" "Resistor_SMD:R_0603_1608Metric"
 			(at 45.72 66.802 90)
 			(effects
@@
 			)
 		)
-		(property "Datasheet" "~"
+		(property "Datasheet" "https://www.lcsc.com/datasheet/lcsc_datasheet_2304140030_YAGEO-RC0603FR-071KL_C22548.pdf"
 			(at 45.72 68.58 0)
 			(effects
@@
 			)
 		)
+		(property "MPN" "RC0603FR-070RL"
+			(at 45.72 68.58 0)
+			(effects
+				(font
+					(size 1.27 1.27)
+				)
+				(hide yes)
+			)
+		)
 		(pin "1"
 		)
@@
 			)
 		)
-		(property "Footprint" "Resistor_SMD:R_0402_1005Metric"
+		(property "Footprint" "Resistor_SMD:R_0603_1608Metric"
 			(at 55.88 38.862 90)
 			(effects
@@
 			)
 		)
-		(property "Datasheet" "~"
+		(property "Datasheet" "https://www.lcsc.com/datasheet/lcsc_datasheet_2304140030_YAGEO-RC0603FR-071KL_C22548.pdf"
 			(at 55.88 40.64 0)
 			(effects
@@
 			)
 		)
+		(property "MPN" "RC0603FR-070RL"
+			(at 55.88 40.64 0)
+			(effects
+				(font
+					(size 1.27 1.27)
+				)
+				(hide yes)
+			)
+		)
 		(pin "1"
 		)
@@
 			)
 		)
-		(property "Footprint" "Inductor_SMD:L_0402_1005Metric"
+		(property "Footprint" "Inductor_SMD:L_0603_1608Metric"
 			(at 118.11 40.64 0)
 			(effects
@@
 			)
 		)
-		(property "Datasheet" "https://search.murata.co.jp/Ceramy/image/img/P02/JELF243B-9117.pdf"
+		(property "Datasheet" "https://www.lcsc.com/datasheet/lcsc_datasheet_2410121551_Taiyo-Yuden-HK16081N8S-T_C222661.pdf"
 			(at 118.11 40.64 0)
 			(effects
@@
 			)
 		)
-		(property "MPN" "LQG15WZ1N8C02D"
+		(property "MPN" "HK16081N8S-T"
 			(at 118.11 40.64 90)
 			(effects
@@
 			)
 		)
+		(property "MPN" "CL10C220JB8NNNC"
+			(at 31.75 46.99 0)
+			(effects
+				(font
+					(size 1.27 1.27)
+				)
+				(hide yes)
+			)
+		)
 		(pin "1"
 		)
@@
 			)
 		)
-		(property "Datasheet" "~"
+		(property "Datasheet" "https://www.lcsc.com/datasheet/lcsc_datasheet_2304140030_YAGEO-RC0603FR-071KL_C22548.pdf"
 			(at 132.08 113.03 0)
 			(effects
@@
 			)
 		)
+		(property "MPN" "RC0603FR-0710KL"
+			(at 132.08 113.03 0)
+			(effects
+				(font
+					(size 1.27 1.27)
+				)
+				(hide yes)
+			)
+		)
 		(pin "1"
 		)
@@
 			)
 		)
+		(property "MPN" "CL10A105KO8NNNC"
+			(at 166.37 63.5 0)
+			(effects
+				(font
+					(size 1.27 1.27)
+				)
+				(hide yes)
+			)
+		)
 		(pin "1"
 		)
@@
 			(at 198.12 114.3 0)
 			(effects
+				(font
+					(size 1.27 1.27)
+				)
+				(hide yes)
+			)
+		)
+		(property "MPN" "CL10B104KO8NNNC"
+			(at 198.12 114.3 0)
+			(effects

Commit message: Release X01-003 - Added "JRM" logo to L3 and and Modem Works logo to L4. - Upated copyright - Added alternates for some components - Some cleanup on SCH and PCB.
Signed-off-by: James Mendel <jrm.mendel@gmail.com>
Parts:
- L1: Alt1 (none) -> BSCH001608081N8S00; Alt2 (none) -> 7447860018; MPN HK16081N8S-T -> LQG18HN1N8S00D
Other:
- company: J. MENDEL -> ${COMPANY}
Changed lines of the file:
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@@
 	(title_block
 		(title "${TITLE}")
-		(date "2025-04-05")
+		(date "2025-04-06")
 		(rev "${REVISION}")
-		(company "J. MENDEL")
+		(company "${COMPANY}")
+		(comment 1 "${LICENSE}")
+		(comment 2 "${COPYRIGHT}")
 	)
 	(rectangle
@@
 	(text_box "Sheet: ${SHEETNAME}"
 		(exclude_from_sim no)
-		(at 177.8 167.64 0)
-		(size 106.68 12.7)
+		(at 213.36 167.64 0)
+		(size 71.12 12.7)
 		(margins 0.9525 0.9525 0.9525 0.9525)
 		(stroke
@@
 					(size 1.27 1.27)
 				)
+				(hide yes)
 			)
 		)
@@
 			)
 		)
-		(property "Datasheet" "https://www.lcsc.com/datasheet/lcsc_datasheet_2410121551_Taiyo-Yuden-HK16081N8S-T_C222661.pdf"
+		(property "Datasheet" "https://search.murata.co.jp/Ceramy/image/img/P02/JELF243B-0002.pdf"
 			(at 118.11 40.64 0)
 			(effects
@@
 			)
 		)
-		(property "MPN" "HK16081N8S-T"
+		(property "MPN" "LQG18HN1N8S00D"
+			(at 118.11 40.64 90)
+			(effects
+				(font
+					(size 1.27 1.27)
+				)
+				(hide yes)
+			)
+		)
+		(property "Alt1" "BSCH001608081N8S00"
+			(at 118.11 40.64 90)
+			(effects
+				(font
+					(size 1.27 1.27)
+				)
+				(hide yes)
+			)
+		)
+		(property "Alt2" "7447860018"
 			(at 118.11 40.64 90)
 			(effects
