File: Power.kicad_sch (KiCad schematic)
At the start: 43 parts, among them J2 S2B-PH-SM4-TB, Q1 DMP3099L, Q2 2N7002, Q3 2N7002, SW4 KMR231NG, SW5 KSS3xxGx, U2 AP2112K-3.3, U3 BQ21040DBV

Commit message: Release X01-004 - Reduced size of 0.3mm pad / 0.2mm pitch to increase pitch to >0.22mm - Removed via-in-pad
Signed-off-by: James Mendel <jrm.mendel@gmail.com>
Parts:
- SW5: Alt1 KSS322GLFG -> KSS331GLFS; Alt2 KSS323GLFG -> KSS351GLFS; MPN KSS312GLFG -> KSS321GLFS
Changed lines of the file:
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@@
 			)
 		)
-		(property "MPN" "KSS312GLFG"
+		(property "MPN" "KSS321GLFS"
 			(at 110.49 60.96 0)
 			(effects
@@
 			)
 		)
-		(property "Alt1" "KSS322GLFG"
+		(property "Alt1" "KSS331GLFS"
 			(at 110.49 60.96 90)
 			(effects
@@
 			)
 		)
-		(property "Alt2" "KSS323GLFG"
+		(property "Alt2" "KSS351GLFS"
 			(at 110.49 60.96 90)
 			(effects
