File: Hardware/Peripherals.kicad_sch (KiCad schematic)
At the start: 15 parts, among them J3 0532610271, J4 Conn_Coaxial, J5 B8B-PH-SM4-TB, U10 PA1616D, U4 DRV2605LDGS, U5 BNO055

Commit message: sch/pb: tweaks for X02-001 release, submit to vendor
Parts:
- J4: now fitted; now in the parts list
- U10: value PA1616D -> ADAFRUIT PA1616D; Alt1 (none) -> 1528-5186-ND; MPN (none) -> 5186
Changed lines of the file:
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@@
 			)
 		)
-		(property "Value" "PA1616D"
+		(property "Value" "ADAFRUIT PA1616D"
 			(at 53.086 35.56 0)
 			(effects
@@
 		(property "Description" "ULTIMATE GPS MODULE PA1616D - 66"
 			(at 77.47 24.13 0)
+			(effects
+				(font
+					(size 1.27 1.27)
+				)
+				(hide yes)
+			)
+		)
+		(property "MPN" "5186"
+			(at 45.72 39.37 0)
+			(effects
+				(font
+					(size 1.27 1.27)
+				)
+				(hide yes)
+			)
+		)
+		(property "Alt1" "1528-5186-ND"
+			(at 45.72 39.37 0)
 			(effects
 				(font
@@
 		(unit 1)
 		(exclude_from_sim no)
-		(in_bom no)
-		(on_board yes)
-		(dnp yes)
+		(in_bom yes)
+		(on_board yes)
+		(dnp no)
 		(property "Reference" "J4"
 			(at 26.924 57.912 0)
