File: Hardware/Peripherals.kicad_sch (KiCad schematic)
At the start: 21 parts, among them J3 0532610271, J5 B8B-PH-SM4-TB, J6 0532610671, U4 DRV2605LDGS, U5 BNO055, U6 M20048-1

Commit message: Sync Hardware from main (hw_X02)
Parts:
- removed C15, C16: 22p, Capacitor_SMD:C_0603_1608Metric, symbol Device:C
- removed J6: 0532610671, Connector_Molex:Molex_PicoBlade_53261-0671_1x06-1MP_P1.25mm_Horizontal, symbol Connector_Generic_MountingPin:Conn_01x06_MountingPin
- removed L1: 1.8n, Inductor_SMD:L_0603_1608Metric, symbol Device:L
- removed R22, R23: 10k, Resistor_SMD:R_0603_1608Metric, symbol Device:R
- removed R24: 0R, Resistor_SMD:R_0603_1608Metric, symbol Device:R
- removed U6: M20048-1, M20048-1:QFN28_M20048-1_ANT, symbol 2025-03-22_21-29-02:M20048-1
- added J4: Conn_Coaxial, Connector_Coaxial:U.FL_Molex_MCRF_73412-0110_Vertical, symbol Connector:Conn_Coaxial
- added U10: ADAFRUIT PA1616D, TESO-LIV3F:PA1616D, symbol 2025-06-15_18-00-59:PA1616D
- C19: value 1u -> 0.1u; MPN CL10A105KO8NNNC -> CL10B104KO8NNNC
Connections:
- net +3.3V: now also U10.1 (VCC)
- net GND: now also J4.2 (Ext), U10.12 (GND), U10.19 (GND), U10.3 (GND), U10.8 (GND)
- net GPS_FIX: now also U10.5 (3D-FIX)
- net GPS_~{RST}: now also U10.2 (NRESET)
- net RX: now also U10.10 (RX0)
- net TX: now also U10.9 (TX0)
- net GPS_VBACKUP renamed GPS_VBAT
- net GPS_VBAT: now also U10.4 (VBACKUP)
- new net: J4.1 (In), U10.11 (EX_ANT)
- no-connect marks 4 -> 12
Other:
- note added: "<10 μA"
- note added: "GPS"
- note removed: "+ Known compatibility + Includes compass"
- note removed: "+ Provides slimmer profile + Price - Locked into this part number"
- note removed: "9600 BAUD"
- note removed: "<30 μA"
- note removed: "Beitian GPS BN-880 Module"
- note removed: "COMPASS HMC5883L ADDR_{(7)} = 0x1E"
- note removed: "GPS Options"
- note removed: "Integrated GPS Module"
- note removed: "Tradeoffs"
- moved on the sheet: J5, R25

Commit message: prepare export for Rev A
Parts:
- J4: now not fitted
Changed lines of the file:
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@@
 	(title_block
 		(title "${TITLE}")
-		(date "2025-08-29")
+		(date "2025-11-18")
 		(rev "${REVISION}")
 		(company "${COMPANY}")
@@
 		(in_bom yes)
 		(on_board yes)
-		(dnp no)
+		(dnp yes)
 		(property "Reference" "J4"
 			(at 26.924 57.912 0)

Commit message: update BOM items to full P/N from previous PCB order feedback
Parts:
- U4: MPN DRV2605LDGS -> DRV2605LDGSR
Changed lines of the file:
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@@
 			)
 		)
-		(property "MPN" "DRV2605LDGS"
+		(property "MPN" "DRV2605LDGSR"
 			(at 53.34 129.54 0)
 			(effects
