File: Hardware/Microcontroller.kicad_sch (KiCad schematic)
At the start: 26 parts, among them J1 GT-USB-7010ASV, SW2 KMR231NG, SW3 KMR231NG, U1 ESP32-S3-MINI-1

Commit message: Sync Hardware from main (hw_X02)
Parts:
- added R23, R24: 100k, Resistor_SMD:R_0603_1608Metric, symbol Device:R
- added TP14: TXD1, M20048-1:TestPoint_Pad_D1.5mm_WITH_LABEL, symbol Connector:TestPoint
- TP12: value TXD0 -> RXD1
Connections:
- net GND: now also R23.2
- net RX: now also TP12.1
- net SPI_MISO: no longer TP12.1
- net TX: now also TP14.1
- net VUSB: now also R24.1
- net BAT_~{CHG}: now reaches U1.32 (SPIIO7/GPIO36/FSPICLK/SUBSPICLK)
- net USB_CONN: now reaches U1.41 (GPIO45)
- net USB_CONN: now also R23.1, R24.2
- net GPS_STBY: no longer names the net of U1.36 (MTDO/GPIO40/CLK_OUT2)
