File: Hardware/Power.kicad_sch (KiCad schematic)
At the start: 43 parts, among them J2 S2B-PH-SM4-TB, Q1 DMP3099L, Q2 2N7002, Q3 2N7002, SW4 KMR231NG, SW5 KSS3xxGx, U2 AP2112K-3.3, U3 BQ21040DBV

Commit message: Sync Hardware from main (hw_X02)
Parts:
- removed Q3: 2N7002, Package_TO_SOT_SMD:SOT-23, symbol Transistor_FET:2N7002
- removed R28, R29: 100k, Resistor_SMD:R_0603_1608Metric, symbol Device:R
- added C21: 0.1u, Capacitor_SMD:C_0603_1608Metric, symbol Device:C
- added D12: B5819WS-TP, Diode_SMD:D_SOD-323, symbol Diode:MBR0520
- added R31: 1.5k, Resistor_SMD:R_0603_1608Metric, symbol Device:R
- added U9: SN74LVC1G14DRL, Package_TO_SOT_SMD:SOT-553, symbol 74xGxx:SN74LVC1G14DRL
- D11, D3, D4: value PMEG2010AEH -> B5819WS-TP; footprint Diode_SMD:D_SOD-123 -> Diode_SMD:D_SOD-323; MPN PMEG2010AEH -> B5819WS-TP
- R11, R14: value 10k -> 100k; MPN RC0603FR-0710KL -> RC0603FR-07100KL
Connections:
- net GND: now also J2.2 (Pin_2), R14.1, C21.2, U9.3 (GND); no longer J2.1 (Pin_1), R14.2
- net SYS_PWROFF: now also R31.1; no longer Q2.1 (G), R13.2
- net VBAT: now also J2.1 (Pin_1); no longer J2.2 (Pin_2)
- net VBAT_MON: now also R14.2; no longer R14.1
- net VUSB: now also D12.1 (K), U9.5 (VCC)
- net at C17.1, R27.2: now also D12.2 (A), U9.2
- net at D11.2 (A), R17.1: now also U9.4
- new net: C21.1, Q2.1 (G), R13.2, R31.2
Other:
- moved on the sheet: J2, R13
