File: Hardware/Terra-HW.kicad_sch (KiCad schematic)
At the start: 7 parts

Commit message: Sync Hardware from main (hw_X02)
Other:
- sheet Microcontroller ports: added BAT_~{CHG}; removed GPS_STBY
- sheet Peripehrals ports: added none; removed GPS_STBY
- sheet Power ports: added BAT_~{CHG}; removed none
